Commit message: modifies invpend urdf

File: invpend_description/urdf/invpend.xacro (robot description, xacro)
@@ -6,5 +6,5 @@
   <xacro:property name="mass" value="1" /> <!-- arbitrary value for mass -->
   <xacro:property name="width" value="0.1" /> <!-- Square dimensions (widthxwidth) of beams -->
-  <xacro:property name="height1" value="2" /> <!-- Link 1 -->
+  <xacro:property name="height1" value="0.1" /> <!-- Link 1 -->
   <xacro:property name="height2" value="1" /> <!-- Link 2 -->
   <xacro:property name="height3" value="1" /> <!-- Link 3 -->
@@ -19,80 +19,75 @@
   <joint name="fixed" type="fixed">
     <parent link="world"/>
-    <child link="link1"/>
+    <child link="slidebar"/>
   </joint>
-  <!-- Base Link -->
-  <link name="link1">
-    <collision>
-      <origin xyz="0 0 ${height1/2}" rpy="0 0 0"/>
+  <!-- Slider Link -->
+  <link name="slidebar">
+    <visual>
+      <origin xyz="0 0 0" rpy="0 0 0"/>
       <geometry>
-	<box size="${width} ${width} ${height1}"/>
-      </geometry>
-    </collision>
-    <visual>
-      <origin xyz="0 0 ${height1/2}" rpy="0 0 0"/>
-      <geometry>
-	<box size="${width} ${width} ${height1}"/>
-      </geometry>
-      <material name="orange"/>
-    </visual>
-    <inertial>
-      <origin xyz="0 0 ${height1/2}" rpy="0 0 0"/>
-      <mass value="${mass}"/>
-      <inertia
-	  ixx="${mass / 12.0 * (width*width + height1*height1)}" ixy="0.0" ixz="0.0"
-	  iyy="${mass / 12.0 * (height1*height1 + width*width)}" iyz="0.0"
-	  izz="${mass / 12.0 * (width*width + width*width)}"/>
-    </inertial>
-  </link>
-  <joint name="joint1" type="continuous">
-    <parent link="link1"/>
-    <child link="link2"/>
-    <origin xyz="0 ${width} ${height1 - axel_offset}" rpy="0 0 0"/>
-    <axis xyz="0 1 0"/>
-    <dynamics damping="0.7"/>
-  </joint>
-  <!-- Middle Link -->
-  <link name="link2">
-    <collision>
-      <origin xyz="0 0 ${height2/2 - axel_offset}" rpy="0 0 0"/>
-      <geometry>
-	<box size="${width} ${width} ${height2}"/>
-      </geometry>
-    </collision>
-    <visual>
-      <origin xyz="0 0 ${height2/2 - axel_offset}" rpy="0 0 0"/>
-      <geometry>
-	<box size="${width} ${width} ${height2}"/>
+	<box size="30 0.05 0.05"/>
       </geometry>
       <material name="black"/>
     </visual>
     <inertial>
-      <origin xyz="0 0 ${height2/2 - axel_offset}" rpy="0 0 0"/>
-      <mass value="${mass}"/>
+      <origin xyz="0 0 0" rpy="0 0 0"/>
+      <mass value="0"/>
       <inertia
-	  ixx="${mass / 12.0 * (width*width + height2*height2)}" ixy="0.0" ixz="0.0"
-	  iyy="${mass / 12.0 * (height2*height2 + width*width)}" iyz="0.0"
-	  izz="${mass / 12.0 * (width*width + width*width)}"/>
+	  ixx="1.0" ixy="0.0" ixz="0.0"
+	  iyy="1.0" iyz="0.0"
+	  izz="1.0"/>
     </inertial>
   </link>
-  <joint name="joint2" type="continuous">
-    <parent link="link2"/>
-    <child link="link3"/>
-    <origin xyz="0 ${width} ${height2 - axel_offset*2}" rpy="0 0 0"/>
-    <axis xyz="0 1 0"/>
-    <dynamics damping="0.7"/>
+  <joint name="slider_to_cart" type="prismatic">
+    <parent link="slidebar"/>
+    <child link="cart"/>
+    <origin xyz="0 0 0" rpy="0 0 0"/>
+    <axis xyz="1 0 0"/>
+    <dynamics damping="0.05"/>
+    <limit effort="1000.0" lower="-15" upper="15" velocity="5"/>
   </joint>
-  <!-- Top Link -->
-  <link name="link3">
+  <!-- Cart Link -->
+  <link name="cart">
     <collision>
-      <origin xyz="0 0 ${height3/2 - axel_offset}" rpy="0 0 0"/>
+      <origin xyz="0 0 0" rpy="0 0 0"/>
       <geometry>
-	<box size="${width} ${width} ${height3}"/>
+	<box size="0.5 0.5 0.2"/>
       </geometry>
     </collision>
     <visual>
-      <origin xyz="0 0 ${height3/2 - axel_offset}" rpy="0 0 0"/>
+      <origin xyz="0 0 0" rpy="0 0 0"/>
       <geometry>
-	<box size="${width} ${width} ${height3}"/>
+	<box size="0.5 0.5 0.2"/>
+      </geometry>
+      <material name="blue"/>
+    </visual>
+    <inertial>
+      <origin xyz="0 0 0" rpy="0 0 0"/>
+      <mass value="1"/>
+      <inertia
+	  ixx="1.0" ixy="0.0" ixz="0.0"
+	  iyy="1.0" iyz="0.0"
+	  izz="1.0"/>
+    </inertial>
+  </link>
+  <joint name="cart_to_pole" type="continuous">
+    <parent link="cart"/>
+    <child link="pole"/>
+    <origin xyz="0 -0.25 0" rpy="0 0 0"/>
+    <axis xyz="0 1 0"/>
+    <dynamics damping="0.5"/>
+  </joint>
+  <!-- Pole Link -->
+  <link name="pole">
+    <collision>
+      <origin xyz="0 0 0.5" rpy="0 0 0"/>
+      <geometry>
+	<box size="0.05 0.05 1"/>
+      </geometry>
+    </collision>
+    <visual>
+      <origin xyz="0 0 0.5" rpy="0 0 0"/>
+      <geometry>
+	<box size="0.05 0.05 1"/>
       </geometry>
       <material name="orange"/>
@@ -100,81 +95,17 @@
     <inertial>
       <origin xyz="0 0 ${height3/2 - axel_offset}" rpy="0 0 0"/>
-      <mass value="${mass}"/>
+      <mass value="10"/>
       <inertia
-	  ixx="${mass / 12.0 * (width*width + height3*height3)}" ixy="0.0" ixz="0.0"
-	  iyy="${mass / 12.0 * (height3*height3 + width*width)}" iyz="0.0"
-	  izz="${mass / 12.0 * (width*width + width*width)}"/>
+	  ixx="1.0" ixy="0.0" ixz="0.0"
+	  iyy="1.0" iyz="0.0"
+	  izz="1.0"/>
     </inertial>
-  </link>
-  <joint name="hokuyo_joint" type="fixed">
-    <axis xyz="0 1 0" />
-    <origin xyz="0 0 ${height3 - axel_offset/2}" rpy="0 0 0"/>
-    <parent link="link3"/>
-    <child link="hokuyo_link"/>
-  </joint>
-  <!-- Hokuyo Laser -->
-  <link name="hokuyo_link">
-    <collision>
-      <origin xyz="0 0 0" rpy="0 0 0"/>
-      <geometry>
-	<box size="0.1 0.1 0.1"/>
-      </geometry>
-    </collision>
-    <visual>
-      <origin xyz="0 0 0" rpy="0 0 0"/>
-      <geometry>
-        <mesh filename="package://invpend_description/meshes/hokuyo.dae"/>
-      </geometry>
-    </visual>
-    <inertial>
-      <mass value="1e-5" />
-      <origin xyz="0 0 0" rpy="0 0 0"/>
-      <inertia ixx="1e-6" ixy="0" ixz="0" iyy="1e-6" iyz="0" izz="1e-6" />
-    </inertial>
-  </link>
-  <joint name="camera_joint" type="fixed">
-    <axis xyz="0 1 0" />
-    <origin xyz="${camera_link} 0 ${height3 - axel_offset*2}" rpy="0 0 0"/>
-    <parent link="link3"/>
-    <child link="camera_link"/>
-  </joint>
-  <!-- Camera -->
-  <link name="camera_link">
-    <collision>
-      <origin xyz="0 0 0" rpy="0 0 0"/>
-      <geometry>
-	<box size="${camera_link} ${camera_link} ${camera_link}"/>
-      </geometry>
-    </collision>
-    <visual>
-      <origin xyz="0 0 0" rpy="0 0 0"/>
-      <geometry>
-	<box size="${camera_link} ${camera_link} ${camera_link}"/>
-      </geometry>
-      <material name="red"/>
-    </visual>
-    <inertial>
-      <mass value="1e-5" />
-      <origin xyz="0 0 0" rpy="0 0 0"/>
-      <inertia ixx="1e-6" ixy="0" ixz="0" iyy="1e-6" iyz="0" izz="1e-6" />
-    </inertial>
-  </link>
-  <!-- generate an optical frame http://www.ros.org/reps/rep-0103.html#suffix-frames
-      so that ros and opencv can operate on the camera frame correctly -->
-  <joint name="camera_optical_joint" type="fixed">
-    <!-- these values have to be these values otherwise the gazebo camera image
-        won't be aligned properly with the frame it is supposedly originating from -->
-    <origin xyz="0 0 0" rpy="${-pi/2} 0 ${-pi/2}"/>
-    <parent link="camera_link"/>
-    <child link="camera_link_optical"/>
-  </joint>
-  <link name="camera_link_optical">
   </link>
   <transmission name="tran1">
     <type>transmission_interface/SimpleTransmission</type>
-    <joint name="joint1">
+    <joint name="slider_to_cart">
       <hardwareInterface>hardware_interface/EffortJointInterface</hardwareInterface>
     </joint>
-    <actuator name="motor1">
+    <actuator name="motor_pris">
       <hardwareInterface>hardware_interface/EffortJointInterface</hardwareInterface>
       <mechanicalReduction>1</mechanicalReduction>
@@ -183,8 +114,8 @@
   <transmission name="tran2">
     <type>transmission_interface/SimpleTransmission</type>
-    <joint name="joint2">
+    <joint name="cart_to_pole">
       <hardwareInterface>hardware_interface/EffortJointInterface</hardwareInterface>
     </joint>
-    <actuator name="motor2">
+    <actuator name="motor_revo">
       <hardwareInterface>hardware_interface/EffortJointInterface</hardwareInterface>
       <mechanicalReduction>1</mechanicalReduction>

Commit message: invpend prototype succeed with position control

File: invpend_description/urdf/invpend.xacro (robot description, xacro)
@@ -24,5 +24,5 @@
   <link name="slidebar">
     <visual>
-      <origin xyz="0 0 0" rpy="0 0 0"/>
+      <origin xyz="0 0 2" rpy="0 0 0"/>
       <geometry>
 	<box size="30 0.05 0.05"/>
@@ -31,6 +31,6 @@
     </visual>
     <inertial>
-      <origin xyz="0 0 0" rpy="0 0 0"/>
-      <mass value="0"/>
+      <origin xyz="0 0 2" rpy="0 0 0"/>
+      <mass value="0.001"/>
       <inertia
 	  ixx="1.0" ixy="0.0" ixz="0.0"
@@ -42,8 +42,8 @@
     <parent link="slidebar"/>
     <child link="cart"/>
-    <origin xyz="0 0 0" rpy="0 0 0"/>
+    <origin xyz="0 0 2" rpy="0 0 0"/>
     <axis xyz="1 0 0"/>
+    <limit effort="1000.0" lower="-15" upper="15" velocity="5"/>
     <dynamics damping="0.05"/>
-    <limit effort="1000.0" lower="-15" upper="15" velocity="5"/>
   </joint>
   <!-- Cart Link -->

Commit message: test velocity control on cart

File: invpend_description/urdf/invpend.xacro (robot description, xacro)
@@ -81,5 +81,5 @@
   <link name="pole">
     <collision>
-      <origin xyz="0 0 0.5" rpy="0 0 0"/>
+      <origin xyz="0 0 -0.5" rpy="0 0 0"/>
       <geometry>
 	<box size="0.05 0.05 1"/>
@@ -87,5 +87,5 @@
     </collision>
     <visual>
-      <origin xyz="0 0 0.5" rpy="0 0 0"/>
+      <origin xyz="0 0 -0.5" rpy="0 0 0"/>
       <geometry>
 	<box size="0.05 0.05 1"/>
@@ -94,5 +94,5 @@
     </visual>
     <inertial>
-      <origin xyz="0 0 ${height3/2 - axel_offset}" rpy="0 0 0"/>
+      <origin xyz="0 0 -0.5" rpy="0 0 0"/>
       <mass value="10"/>
       <inertia

Commit message: code gazebo usable q-learning

File: invpend_description/urdf/invpend.xacro (robot description, xacro)
@@ -26,5 +26,5 @@
       <origin xyz="0 0 2" rpy="0 0 0"/>
       <geometry>
-	<box size="30 0.05 0.05"/>
+	<box size="10 0.05 0.05"/>
       </geometry>
       <material name="black"/>
@@ -44,6 +44,6 @@
     <origin xyz="0 0 2" rpy="0 0 0"/>
     <axis xyz="1 0 0"/>
-    <limit effort="1000.0" lower="-15" upper="15" velocity="5"/>
-    <dynamics damping="0.05"/>
+    <limit effort="1000.0" lower="-5" upper="5" velocity="5"/>
+    <dynamics damping="0.01"/>
   </joint>
   <!-- Cart Link -->
@@ -76,5 +76,5 @@
     <origin xyz="0 -0.25 0" rpy="0 0 0"/>
     <axis xyz="0 1 0"/>
-    <dynamics damping="0.5"/>
+    <dynamics damping="0.01"/>
   </joint>
   <!-- Pole Link -->
@@ -95,5 +95,5 @@
     <inertial>
       <origin xyz="0 0 -0.5" rpy="0 0 0"/>
-      <mass value="10"/>
+      <mass value="0.5"/>
       <inertia
 	  ixx="1.0" ixy="0.0" ixz="0.0"

Commit message: ros_control keeps pole upright

File: invpend_description/urdf/invpend.xacro (robot description, xacro)
@@ -44,6 +44,6 @@
     <origin xyz="0 0 2" rpy="0 0 0"/>
     <axis xyz="1 0 0"/>
-    <limit effort="1000.0" lower="-5" upper="5" velocity="5"/>
-    <dynamics damping="0.01"/>
+    <limit effort="1000.0" lower="-5" upper="5" velocity="10"/>
+    <dynamics damping="0.001"/>
   </joint>
   <!-- Cart Link -->
@@ -81,5 +81,5 @@
   <link name="pole">
     <collision>
-      <origin xyz="0 0 -0.5" rpy="0 0 0"/>
+      <origin xyz="0 0 0.5" rpy="0 0 0"/>
       <geometry>
 	<box size="0.05 0.05 1"/>
@@ -87,5 +87,5 @@
     </collision>
     <visual>
-      <origin xyz="0 0 -0.5" rpy="0 0 0"/>
+      <origin xyz="0 0 0.5" rpy="0 0 0"/>
       <geometry>
 	<box size="0.05 0.05 1"/>
@@ -94,6 +94,6 @@
     </visual>
     <inertial>
-      <origin xyz="0 0 -0.5" rpy="0 0 0"/>
-      <mass value="0.5"/>
+      <origin xyz="0 0 0.5" rpy="0 0 0"/>
+      <mass value="2"/>
       <inertia
 	  ixx="1.0" ixy="0.0" ixz="0.0"

Commit message: fix cart_to_pole control issue

File: invpend_description/urdf/invpend.xacro (robot description, xacro)
@@ -32,5 +32,5 @@
     <inertial>
       <origin xyz="0 0 2" rpy="0 0 0"/>
-      <mass value="0.001"/>
+      <mass value="100"/>
       <inertia
 	  ixx="1.0" ixy="0.0" ixz="0.0"
@@ -45,5 +45,5 @@
     <axis xyz="1 0 0"/>
     <limit effort="1000.0" lower="-5" upper="5" velocity="10"/>
-    <dynamics damping="0.001"/>
+    <dynamics damping="0.01"/>
   </joint>
   <!-- Cart Link -->
@@ -76,5 +76,5 @@
     <origin xyz="0 -0.25 0" rpy="0 0 0"/>
     <axis xyz="0 1 0"/>
-    <dynamics damping="0.01"/>
+    <dynamics damping="0.001"/>
   </joint>
   <!-- Pole Link -->
@@ -95,5 +95,5 @@
     <inertial>
       <origin xyz="0 0 0.5" rpy="0 0 0"/>
-      <mass value="2"/>
+      <mass value="5"/>
       <inertia
 	  ixx="1.0" ixy="0.0" ixz="0.0"

Commit message: minor change on model urdf

File: invpend_description/urdf/invpend.xacro (robot description, xacro)
@@ -44,5 +44,5 @@
     <origin xyz="0 0 2" rpy="0 0 0"/>
     <axis xyz="1 0 0"/>
-    <limit effort="1000.0" lower="-5" upper="5" velocity="10"/>
+    <limit effort="1000.0" lower="-5" upper="5" velocity="100"/>
     <dynamics damping="0.01"/>
   </joint>
@@ -95,5 +95,5 @@
     <inertial>
       <origin xyz="0 0 0.5" rpy="0 0 0"/>
-      <mass value="5"/>
+      <mass value="3"/>
       <inertia
 	  ixx="1.0" ixy="0.0" ixz="0.0"

Commit message: change reset strategy to pub set_link_state topic

File: invpend_description/urdf/invpend.xacro (robot description, xacro)
@@ -32,5 +32,5 @@
     <inertial>
       <origin xyz="0 0 2" rpy="0 0 0"/>
-      <mass value="100"/>
+      <mass value="1000"/>
       <inertia
 	  ixx="1.0" ixy="0.0" ixz="0.0"

Commit message: modify reference frame for slidebar in urdf

File: invpend_description/urdf/invpend.xacro (robot description, xacro)
@@ -20,9 +20,10 @@
     <parent link="world"/>
     <child link="slidebar"/>
+    <origin xyz="0 0 2"/>
   </joint>
   <!-- Slider Link -->
   <link name="slidebar">
     <visual>
-      <origin xyz="0 0 2" rpy="0 0 0"/>
+      <origin xyz="0 0 0" rpy="0 0 0"/>
       <geometry>
 	<box size="10 0.05 0.05"/>
@@ -31,5 +32,5 @@
     </visual>
     <inertial>
-      <origin xyz="0 0 2" rpy="0 0 0"/>
+      <origin xyz="0 0 0" rpy="0 0 0"/>
       <mass value="1000"/>
       <inertia
@@ -42,5 +43,5 @@
     <parent link="slidebar"/>
     <child link="cart"/>
-    <origin xyz="0 0 2" rpy="0 0 0"/>
+    <origin xyz="0 0 0" rpy="0 0 0"/>
     <axis xyz="1 0 0"/>
     <limit effort="1000.0" lower="-5" upper="5" velocity="100"/>
@@ -66,7 +67,7 @@
       <mass value="1"/>
       <inertia
-	  ixx="1.0" ixy="0.0" ixz="0.0"
-	  iyy="1.0" iyz="0.0"
-	  izz="1.0"/>
+	  ixx="0.001" ixy="0.0" ixz="0.0"
+	  iyy="0.001" iyz="0.0"
+	  izz="0.001"/>
     </inertial>
   </link>
@@ -74,5 +75,5 @@
     <parent link="cart"/>
     <child link="pole"/>
-    <origin xyz="0 -0.25 0" rpy="0 0 0"/>
+    <origin xyz="0 -0.255 0" rpy="0 0 0"/>
     <axis xyz="0 1 0"/>
     <dynamics damping="0.001"/>
@@ -97,7 +98,7 @@
       <mass value="3"/>
       <inertia
-	  ixx="1.0" ixy="0.0" ixz="0.0"
-	  iyy="1.0" iyz="0.0"
-	  izz="1.0"/>
+	  ixx="0.001" ixy="0.0" ixz="0.0"
+	  iyy="0.001" iyz="0.0"
+	  izz="0.001"/>
     </inertial>
   </link>

Commit message: modify env reset parameters, fails to reset

File: invpend_description/urdf/invpend.xacro (robot description, xacro)
@@ -75,5 +75,5 @@
     <parent link="cart"/>
     <child link="pole"/>
-    <origin xyz="0 -0.255 0" rpy="0 0 0"/>
+    <origin xyz="0 -0.275 0" rpy="0 0 0"/>
     <axis xyz="0 1 0"/>
     <dynamics damping="0.001"/>

Commit message: modify cartpole model, correspond to openAI gym; continue for gazebo and joint control

File: invpend_description/urdf/invpend.xacro (robot description, xacro)
@@ -4,11 +4,13 @@
   <!-- Constants for robot dimensions -->
   <xacro:property name="PI" value="3.1415926535897931"/>
-  <xacro:property name="mass" value="1" /> <!-- arbitrary value for mass -->
-  <xacro:property name="width" value="0.1" /> <!-- Square dimensions (widthxwidth) of beams -->
-  <xacro:property name="height1" value="0.1" /> <!-- Link 1 -->
-  <xacro:property name="height2" value="1" /> <!-- Link 2 -->
-  <xacro:property name="height3" value="1" /> <!-- Link 3 -->
-  <xacro:property name="camera_link" value="0.05" /> <!-- Size of square 'camera' box -->
-  <xacro:property name="axel_offset" value="0.05" /> <!-- Space btw top of beam and the each joint -->
+  <xacro:property name="mass_slider" value="100" /> <!-- arbitrary value for mass -->
+  <xacro:property name="mass_cart" value="1.0" /> <!-- arbitrary value for mass -->
+  <xacro:property name="mass_pole" value="0.1" /> <!-- arbitrary value for mass -->
+  <xacro:property name="width" value="0.25" /> <!-- cart width -->
+  <xacro:property name="height" value="0.2" /> <!-- cart height -->
+  <xacro:property name="depth" value="0.25" /> <!-- cart depth -->
+  <xacro:property name="length_slider" value="5" /> <!-- pole length -->
+  <xacro:property name="length_pole" value="0.5" /> <!-- pole length -->
+  <xacro:property name="radius" value="0.05" /> <!-- slender bar radius -->
   <!-- Import all Gazebo-customization elements, including Gazebo colors -->
   <xacro:include filename="$(find invpend_description)/urdf/invpend.gazebo" />
@@ -27,5 +29,5 @@
       <origin xyz="0 0 0" rpy="0 0 0"/>
       <geometry>
-	<box size="10 0.05 0.05"/>
+	<box size="${length_slider} ${radius} ${radius}"/>
       </geometry>
       <material name="black"/>
@@ -33,9 +35,9 @@
     <inertial>
       <origin xyz="0 0 0" rpy="0 0 0"/>
-      <mass value="1000"/>
+      <mass value="${mass_slider}"/>
       <inertia
-	  ixx="1.0" ixy="0.0" ixz="0.0"
-	  iyy="1.0" iyz="0.0"
-	  izz="1.0"/>
+	  ixx="${mass_slider*length_slider*length_slider/12}" ixy="0.0" ixz="0.0"
+	  iyy="0.0" iyz="0.0"
+	  izz="${mass_slider*length_slider*length_slider/12}"/>
     </inertial>
   </link>
@@ -45,6 +47,6 @@
     <origin xyz="0 0 0" rpy="0 0 0"/>
     <axis xyz="1 0 0"/>
-    <limit effort="1000.0" lower="-5" upper="5" velocity="100"/>
-    <dynamics damping="0.01"/>
+    <limit effort="100.0" lower="-2.5" upper="2.5" velocity="1000"/>
+    <dynamics damping="0.0001"/>
   </joint>
   <!-- Cart Link -->
@@ -53,5 +55,5 @@
       <origin xyz="0 0 0" rpy="0 0 0"/>
       <geometry>
-	<box size="0.5 0.5 0.2"/>
+	<box size="${width} ${depth} ${height}"/>
       </geometry>
     </collision>
@@ -59,5 +61,5 @@
       <origin xyz="0 0 0" rpy="0 0 0"/>
       <geometry>
-	<box size="0.5 0.5 0.2"/>
+	<box size="${width} ${depth} ${height}"/>
       </geometry>
       <material name="blue"/>
@@ -65,40 +67,40 @@
     <inertial>
       <origin xyz="0 0 0" rpy="0 0 0"/>
-      <mass value="1"/>
+      <mass value="${mass_cart}"/>
       <inertia
-	  ixx="0.001" ixy="0.0" ixz="0.0"
-	  iyy="0.001" iyz="0.0"
-	  izz="0.001"/>
+	  ixx="${mass_cart*(depth*depth+height*height)/12}" ixy="0.0" ixz="0.0"
+	  iyy="${mass_cart*(depth*depth+width*width)/12}" iyz="0.0"
+	  izz="${mass_cart*(width*width+height*height)/12}"/>
     </inertial>
   </link>
-  <joint name="cart_to_pole" type="continuous">
+  <joint name="cart_to_pole" type="revolute">
     <parent link="cart"/>
     <child link="pole"/>
-    <origin xyz="0 -0.275 0" rpy="0 0 0"/>
+    <origin xyz="0 -0.15 0" rpy="0 0 0"/>
     <axis xyz="0 1 0"/>
-    <dynamics damping="0.001"/>
+    <limit effort="1000.0" lower="${-PI}" upper = "${PI}" velocity="1000.0"/>
   </joint>
   <!-- Pole Link -->
   <link name="pole">
     <collision>
-      <origin xyz="0 0 0.5" rpy="0 0 0"/>
+      <origin xyz="0 0 0.25" rpy="0 0 0"/>
       <geometry>
-	<box size="0.05 0.05 1"/>
+	<box size="${radius} ${radius} ${length_pole}"/>
       </geometry>
     </collision>
     <visual>
-      <origin xyz="0 0 0.5" rpy="0 0 0"/>
+      <origin xyz="0 0 0.25" rpy="0 0 0"/>
       <geometry>
-	<box size="0.05 0.05 1"/>
+	<box size="${radius} ${radius} ${length_pole}"/>
       </geometry>
       <material name="orange"/>
     </visual>
     <inertial>
-      <origin xyz="0 0 0.5" rpy="0 0 0"/>
-      <mass value="3"/>
+      <origin xyz="0 0 0.25" rpy="0 0 0"/>
+      <mass value="${mass_pole}"/>
       <inertia
-	  ixx="0.001" ixy="0.0" ixz="0.0"
-	  iyy="0.001" iyz="0.0"
-	  izz="0.001"/>
+	  ixx="${mass_pole*length_pole*length_pole/3}" ixy="0.0" ixz="0.0"
+	  iyy="0.0" iyz="0.0"
+	  izz="${mass_pole*length_pole*length_pole/3}"/>
     </inertial>
   </link>
