Commit message: update cart-pole model urdf, cannot use openAI mass setting

File: invpend_description/urdf/invpend.xacro (robot description, xacro)
@@ -5,12 +5,13 @@
   <xacro:property name="PI" value="3.1415926535897931"/>
   <xacro:property name="mass_slider" value="100" /> <!-- arbitrary value for mass -->
-  <xacro:property name="mass_cart" value="1.0" /> <!-- arbitrary value for mass -->
-  <xacro:property name="mass_pole" value="0.1" /> <!-- arbitrary value for mass -->
+  <xacro:property name="mass_cart" value="20.0" /> <!-- arbitrary value for mass -->
+  <xacro:property name="mass_pole" value="2.0" /> <!-- arbitrary value for mass -->
   <xacro:property name="width" value="0.25" /> <!-- cart width -->
-  <xacro:property name="height" value="0.2" /> <!-- cart height -->
+  <xacro:property name="height" value="0.125" /> <!-- cart height -->
   <xacro:property name="depth" value="0.25" /> <!-- cart depth -->
   <xacro:property name="length_slider" value="5" /> <!-- pole length -->
   <xacro:property name="length_pole" value="0.5" /> <!-- pole length -->
-  <xacro:property name="radius" value="0.05" /> <!-- slender bar radius -->
+  <xacro:property name="radius" value="0.01" /> <!-- slender bar radius -->
+  <xacro:property name="radius_pole" value="0.025" /> <!-- pole radius -->
   <!-- Import all Gazebo-customization elements, including Gazebo colors -->
   <xacro:include filename="$(find invpend_description)/urdf/invpend.gazebo" />
@@ -22,5 +23,5 @@
     <parent link="world"/>
     <child link="slidebar"/>
-    <origin xyz="0 0 2"/>
+    <origin xyz="0 0 1"/>
   </joint>
   <!-- Slider Link -->
@@ -48,5 +49,5 @@
     <axis xyz="1 0 0"/>
     <limit effort="100.0" lower="-2.5" upper="2.5" velocity="1000"/>
-    <dynamics damping="0.0001"/>
+    <!--dynamics damping="0.0001"/-->
   </joint>
   <!-- Cart Link -->
@@ -77,5 +78,5 @@
     <parent link="cart"/>
     <child link="pole"/>
-    <origin xyz="0 -0.15 0" rpy="0 0 0"/>
+    <origin xyz="0 ${-depth/2-radius-radius_pole/2} ${height/4}" rpy="0 0 0"/>
     <axis xyz="0 1 0"/>
     <limit effort="1000.0" lower="${-PI}" upper = "${PI}" velocity="1000.0"/>
@@ -84,18 +85,18 @@
   <link name="pole">
     <collision>
-      <origin xyz="0 0 0.25" rpy="0 0 0"/>
+      <origin xyz="0 0 ${length_pole/2}" rpy="0 0 0"/>
       <geometry>
-	<box size="${radius} ${radius} ${length_pole}"/>
+	<box size="${radius_pole} ${radius_pole} ${length_pole}"/>
       </geometry>
     </collision>
     <visual>
-      <origin xyz="0 0 0.25" rpy="0 0 0"/>
+      <origin xyz="0 0 ${length_pole/2}" rpy="0 0 0"/>
       <geometry>
-	<box size="${radius} ${radius} ${length_pole}"/>
+	<box size="${radius_pole} ${radius_pole} ${length_pole}"/>
       </geometry>
       <material name="orange"/>
     </visual>
     <inertial>
-      <origin xyz="0 0 0.25" rpy="0 0 0"/>
+      <origin xyz="0 0 ${length_pole/2}" rpy="0 0 0"/>
       <mass value="${mass_pole}"/>
       <inertia
